File: left.kicad_sch (KiCad schematic)
At the start: 139 parts, among them J2 USB_C_Receptacle_USB2.0_16P, J5 Conn_01x05, J7 Battery, Q3 AO3401A, Q5 2N7002, Q6 AO3401A, SW4 RST, SW7 PWR, SW8 RotaryEncoder_Switch, U10 TP4056, U4 PRTR5V0U2X, U5 nRF52840_holyiot_18010, U7 XC6206PxxxMR

Commit message: finished routing, need to review
Parts:
- removed J5: Conn_01x05, Connector_IDC:IDC-Header_2x03_P2.54mm_Vertical_SMD, symbol Connector_Generic:Conn_01x05
- added J1: wurth_6_pin_SKEDD, 490107670612:wurth_6_pin_SKEDD, symbol Wurth_6_pin_Connector:wurth_6_pin_SKEDD
- D1, D10, D11, D12, D13, D14, D15, D16, D17, D18, D19, D2, D20, D21, D22, D23, D24, D25, D26, D27, D28, D3, D4, D5, D6, D7, D8, D9: footprint reversible_skyline:designator_swapped_D_0805_2012Metric_Pad1.15x1.40mm_HandSolder -> Diode_SMD:D_0805_2012Metric_Pad1.15x1.40mm_HandSolder
- MH1: value MountingHole -> MH1; footprint (none) -> reversible_skyline:mounting_hole_npth
- MH2: value MountingHole -> MH2; footprint (none) -> reversible_skyline:mounting_hole_npth
- MH3: value MountingHole -> MH3; footprint (none) -> reversible_skyline:mounting_hole_npth
- MH4: value MountingHole -> MH4; footprint (none) -> reversible_skyline:mounting_hole_npth
- MH5: value MountingHole -> MH5; footprint (none) -> reversible_skyline:mounting_hole_npth
Connections:
- net +3.3V: now also J1.1
- net COL0: now also U5.7 (P0.02-LF-A); no longer U5.30 (P1.02-LF)
- net COL1: now also U5.8 (P0.28-LF-A); no longer U5.29 (P1.01-LF)
- net COL2: now also U5.9 (P0.29-LF-A); no longer U5.28 (P1.03-LF)
- net COL3: now also U5.10 (P0.30-LF-A); no longer U5.27 (P1.00)
- net COL4: now also U5.11 (P0.31-LF-A); no longer U5.26 (P0.22)
- net COL5: now also U5.12 (P0.04-A); no longer U5.20 (P0.19)
- net CS: now also U5.19 (P0.21); no longer U5.4 (P1.13-LF)
- net EncoderTermA: now also U5.30 (P1.02-LF); no longer U5.18 (P0.23)
- net EncoderTermB: now also U5.29 (P1.01-LF); no longer U5.19 (P0.21)
- net GND: now also J1.5
- net LED_Ctrl: now also U5.28 (P1.03-LF); no longer U5.5 (P1.15-LF)
- net MOSI: now also U5.17 (P0.12); no longer U5.33 (P1.04-LF)
- net ROW0: now also U5.2 (P1.11-LF); no longer U5.6 (P0.03-LF-A)
- net ROW1: now also U5.3 (P1.10-LF); no longer U5.7 (P0.02-LF-A)
- net ROW2: now also U5.4 (P1.13-LF); no longer U5.8 (P0.28-LF-A)
- net ROW3: now also U5.5 (P1.15-LF); no longer U5.9 (P0.29-LF-A)
- net ROW4: now also U5.6 (P0.03-LF-A); no longer U5.10 (P0.30-LF-A)
- net RST: now also J1.3
- net SCK: now also U5.18 (P0.23); no longer U5.34 (P1.06-LF)
- net SWDCLK: now also J1.4
- net SWDIO: now also J1.2
- net Vsense: now also U5.26 (P0.22); no longer U5.11 (P0.31-LF-A)
- net Vsense_EN: now also U5.27 (P1.00); no longer U5.12 (P0.04-A)
- no-connect marks 30 -> 31
