File: right.kicad_sch (KiCad schematic)
At the start: 122 parts, among them J3 USB_C_Receptacle_USB2.0_16P, J6 Conn_01x05, J8 Battery, Q4 AO3401A, Q7 2N7002, Q8 AO3401A, SW10 RotaryEncoder_Switch, SW5 RST, SW9 PWR, U11 TP4056, U6 PRTR5V0U2X, U8 XC6206PxxxMR, U9 nRF52840_holyiot_18010

Commit message: finished routing, need to review
Parts:
- removed C10: 4u7, Capacitor_SMD:C_0402_1005Metric, symbol Device:C_Small
- removed C17, C20: 1u, Capacitor_SMD:C_0402_1005Metric, symbol Device:C_Small
- removed C18, C21, C38, C39: 0.1u, Capacitor_SMD:C_0402_1005Metric, symbol Device:C_Small
- removed C22, C9: 10u, symbol Device:C_Polarized_Small
- removed C23: 0.1uF, Capacitor_SMD:C_0402_1005Metric, symbol Device:C
- removed D29, D49, D50, D51, D52, D53, D54, D55, D58, D59, D60, D61, D62, D67, D68, D69, D70, D71, D76, D77, D78, D79, D80, D83, D86, D87, D88, D89: D_Small, Diode_SMD:D_0805_2012Metric_Pad1.15x1.40mm_HandSolder, symbol Device:D_Small
- removed D32: orange, LED_SMD:LED_0402_1005Metric_Pad0.77x0.64mm_HandSolder, symbol Device:LED_Small
- removed D48: Schottky, symbol Device:D_Schottky
- removed D56, D57, D63, D64, D65, D66, D72, D73, D74, D75, D81, D82, D84: LED, Diode_SMD:D_0805_2012Metric_Pad1.15x1.40mm_HandSolder, symbol Device:LED
- removed F3: 500mA, Fuse:Fuse_1206_3216Metric, symbol Device:Polyfuse
- removed J3: USB_C_Receptacle_USB2.0_16P, PCM_marbastlib-various:USB_C_Receptacle_HRO_TYPE-C-31-M-12, symbol Connector:USB_C_Receptacle_USB2.0_16P
- removed J6: Conn_01x05, Connector_PinHeader_2.54mm:PinHeader_1x05_P2.54mm_Horizontal, symbol Connector_Generic:Conn_01x05
- removed J8: Battery, PCM_marbastlib-various:Molex_Pico-EZmate_78171-0002_1x02-1MP_P1.20mm_Vertical, symbol Connector_Generic_MountingPin:Conn_01x02_MountingPin
- removed Q4, Q8: AO3401A, Package_TO_SOT_SMD:SOT-23, symbol Transistor_FET:AO3401A
- removed Q7: 2N7002, Package_TO_SOT_SMD:SOT-23, symbol Transistor_FET:2N7002
- removed R10, R34: 1k5, Resistor_SMD:R_0805_2012Metric_Pad1.20x1.40mm_HandSolder, symbol Device:R_Small
- removed R26, R32: 5.1k, Resistor_SMD:R_0805_2012Metric_Pad1.20x1.40mm_HandSolder, symbol Device:R
- removed R33: 5k, Resistor_SMD:R_0805_2012Metric_Pad1.20x1.40mm_HandSolder, symbol Device:R_Small
- removed R35, R38: 0R, Resistor_SMD:R_0805_2012Metric_Pad1.20x1.40mm_HandSolder, symbol Device:R
- removed R36: 806k, Resistor_SMD:R_0805_2012Metric_Pad1.20x1.40mm_HandSolder, symbol Device:R_Small
- removed R37: 2M, Resistor_SMD:R_0805_2012Metric_Pad1.20x1.40mm_HandSolder, symbol Device:R_Small
- removed R39, R40, R41, R42, R43, R44, R45, R46, R47, R48, R49, R50, R51: 1.5k, Resistor_SMD:R_0805_2012Metric_Pad1.20x1.40mm_HandSolder, symbol Device:R
- removed R54: 47, Resistor_SMD:R_0805_2012Metric_Pad1.20x1.40mm_HandSolder, symbol Device:R
- removed R55, R57: 5k, Resistor_SMD:R_0805_2012Metric_Pad1.20x1.40mm_HandSolder, symbol Device:R
- removed R56, R58: 10k, Resistor_SMD:R_0805_2012Metric_Pad1.20x1.40mm_HandSolder, symbol Device:R_Small
- removed S29, S30, S31, S32, S33, S34, S35, S36, S37, S38, S39, S40, S41, S42, S43, S44, S45, S46, S47, S48, S49, S50, S51, S52, S53, S54, S55, S56: MX_SW_solder, symbol PCM_marbastlib-mx:MX_SW_solder
- removed SW10: RotaryEncoder_Switch, symbol Device:RotaryEncoder_Switch
- removed SW5: RST, PCM_marbastlib-various:SW_SPST_SKQG_WithStem, symbol Switch:SW_Push_45deg
- removed SW9: PWR, PCM_marbastlib-various:SW_MSK12C02-HB, symbol Switch:SW_Push_SPDT
- removed U11: TP4056, reversible_skyline:TP4056_reversible, symbol PCM_marbastlib-various:TP4056
- removed U6: PRTR5V0U2X, Package_TO_SOT_SMD:SOT-143, symbol Power_Protection:PRTR5V0U2X
- removed U8: XC6206PxxxMR, Package_TO_SOT_SMD:SOT-23, symbol Regulator_Linear:XC6206PxxxMR
- removed U9: nRF52840_holyiot_18010, PCM_marbastlib-various:nRF52840_holyiot_18010, symbol PCM_marbastlib-various:nRF52840_holyiot_18010
Connections:
- no-connect marks 32 -> 0
Other:
- note removed: "" '"
- note removed: "0"
- note removed: "1"
- note removed: "2"
- note removed: "3"
- note removed: "4"
- note removed: "5"
- note removed: "6"
- note removed: "7"
- note removed: "8"
- note removed: "9"
- note removed: ": ;"
- note removed: "< ,"
- note removed: "> ."
- note removed: "? /"
- note removed: "A"
- note removed: "Alt"
- note removed: "B"
- note removed: "Battery"
- note removed: "Bck"
- note removed: "C"
- note removed: "Col0"
- note removed: "Col1"
- note removed: "Col2"
- note removed: "Col3"
- note removed: "Col4"
- note removed: "Col5"
- note removed: "Ctrl"
- note removed: "Current draw: 1mA*14=0.14A"
- note removed: "D"
- note removed: "E"
- note removed: "Enc"
- note removed: "Ent"
- note removed: "Esc"
- note removed: "Extra switch footprint"
- note removed: "F"
- note removed: "FN"
- note removed: "G"
- note removed: "H"
- note removed: "I"
- note removed: "J"
- note removed: "K"
- note removed: "L"
- note removed: "LCD"
- note removed: "Left"
- note removed: "M"
- note removed: "MCU"
- note removed: "N"
- note removed: "No encoder footprints for right side (encoder can be connected flipped)"
- note removed: "No switch footprints for right side (left side has reversible footprints)"
- note removed: "O"
- note removed: "P"
- note removed: "PROG: 5 kOhm -> 250 mA charging current TEMP: Pulled to GND -> no OTP"
- note removed: "Pin header for ST-Link to connect and flash bootloader"
- note removed: "Q"
- note removed: "R"
- note removed: "Resistor Value: (Vf-Vd)/I =(5-3.2)/1mA =1.8kohm ≈1.5kohm (BOM optimization)"
- note removed: "Right"
- note removed: "Row0"
- note removed: "Row1"
- note removed: "Row2"
- note removed: "Row3"
- note removed: "Row4"
- note removed: "S"
- note removed: "Shift"
- note removed: "Spc"
- note removed: "Switch Matrix"
- note removed: "T"
- note removed: "Tab"
- note removed: "U"
- note removed: "USB-C"
- note removed: "V"
- note removed: "W"
- note removed: "White Underglow"
- note removed: "Win"
- note removed: "X"
- note removed: "Y"
- note removed: "Z"
- note removed: "disconnects load while charging"
- note removed: "not sure how to implement this in zmk yet, solder r to gnd for backup if vsens_en doesnt work"
- note removed: "resistor value could be 5k for bom optimization"
- note removed: "| \"
