File: skyline.kicad_pcb (KiCad board)
At the start: 2 copper layers, 140.5 x 109.7 mm, 158 parts, among them J7 Battery, Q3 AO3401A, Q5 2N7002, Q6 AO3401A, SW4 RST, SW7 PWR, SW8 RotaryEncoder_Switch, U10 TP4056, U11 TXB0101, U4 PRTR5V0U2X, U5 nRF52840_holyiot_18010, U7 XC6206PxxxMR

Commit message: Added rev. led footprints, jumpers for niceview
Parts:
- removed B1: , E73:SW_TACT_ALPS_SKQGABE010
- removed C20, C21, C22, C23, C24, C25, C26, C27, C28, C29, C30, C31, C32, C33, C34, C35: 0.1 uF, Capacitor_SMD:C_0402_1005Metric_Pad0.74x0.62mm_HandSolder
- removed D71, D72, D73, D74, D75, D76, D77, D78, D79, D80, D81, D82, D83, D84: WS2812B, LED_SMD:LED_WS2812B_PLCC4_5.0x5.0mm_P3.2mm
- removed U11: TXB0101, Package_TO_SOT_SMD:SOT-363_SC-70-6_Handsoldering
- added C16: 0.1u, Capacitor_SMD:C_0402_1005Metric, F.Cu at (344.3, 124.2)
- added J5: Conn_01x05, Connector_PinHeader_2.54mm:PinHeader_1x05_P2.54mm_Vertical, F.Cu at (311.5, 142.4)
- added JP1: SolderJumper_2_Open, reversible_skyline:Jumper_solder, F.Cu at (285.8, 103.3)
- added JP10: SolderJumper_2_Open, reversible_skyline:Jumper_solder, F.Cu at (289.2, 115.0)
- added JP2: SolderJumper_2_Open, reversible_skyline:Jumper_solder, F.Cu at (285.8, 106.2)
- added JP3: SolderJumper_2_Open, reversible_skyline:Jumper_solder, F.Cu at (285.8, 109.2)
- added JP4: SolderJumper_2_Open, reversible_skyline:Jumper_solder, F.Cu at (285.8, 112.1)
- added JP5: SolderJumper_2_Open, reversible_skyline:Jumper_solder, F.Cu at (285.8, 115.0)
- added JP6: SolderJumper_2_Open, reversible_skyline:Jumper_solder, F.Cu at (289.2, 103.3)
- added JP7: SolderJumper_2_Open, reversible_skyline:Jumper_solder, F.Cu at (289.2, 106.2)
- added JP8: SolderJumper_2_Open, reversible_skyline:Jumper_solder, F.Cu at (289.2, 109.2)
- added JP9: SolderJumper_2_Open, reversible_skyline:Jumper_solder, F.Cu at (289.2, 112.1)
- D1, D10, D11, D12, D13, D14, D15, D16, D17, D18, D19, D2, D20, D21, D22, D23, D24, D25, D26, D27, D28, D3, D4, D5, D6, D7, D8, D9: footprint Diode_SMD:D_0805_2012Metric_Pad1.15x1.40mm_HandSolder -> reversible_skyline:reversible_D_0805_2012Metric_Pad1.15x1.40mm_HandSolder
- D33, D34, D35, D36, D37, D38, D39, D40, D41, D42, D43, D44, D45, D46, D47: footprint LED_THT:LED_D5.0mm -> reversible_skyline:reversible_D_0805_2012Metric_Pad1.15x1.40mm_HandSolder
- OLED1: footprint lib:OLED_headers -> nice_view:nice_view
- S1, S10, S11, S12, S13, S14, S15, S16, S17, S18, S19, S2, S20, S21, S22, S23, S24, S25, S26, S27, S28, S3, S4, S5, S6, S7, S8, S9: footprint PG1350 -> PCM_marbastlib-xp-choc:SW_choc_Reversible_1u
- moved OLED1 104.2 mm to (302.5, 36.2), turned to 0 degrees
- moved SW8 64.9 mm to (261.0, 139.5)
- moved D45 58.1 mm to (322.9, 102.3)
- moved D46 57.4 mm to (322.9, 104.9)
- moved D47 57.1 mm to (322.9, 107.5)
- moved D42 56.3 mm to (318.5, 107.5)
- moved D44 50.0 mm to (322.9, 99.8)
- moved D43 49.6 mm to (322.9, 97.2)
- moved D39 47.2 mm to (318.5, 99.8)
- moved D40 46.6 mm to (318.5, 102.3)
- moved D41 46.5 mm to (318.5, 104.9)
- moved D36 45.5 mm to (314.1, 104.9)
- moved D37 44.3 mm to (314.1, 107.5)
- moved D38 40.0 mm to (318.5, 97.2)
- moved U5 37.9 mm to (288.5, 88.2)
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Connections:
- OLED1 pad 1: MOSI -> Net-(JP1-B)
- OLED1 pad 2: SCK -> Net-(JP2-B)
- OLED1 pad 3: +3.3V -> Net-(JP3-B)
- OLED1 pad 4: Case -> Net-(JP4-B)
Other:
- outline, holes or cut-outs redrawn

Commit message: finished routing, need to fix it up now
Parts:
- removed D32: green, LED_SMD:LED_0402_1005Metric_Pad0.77x0.64mm_HandSolder
- removed D46, D47: LED, reversible_skyline:reversible_D_0805_2012Metric_Pad1.15x1.40mm_HandSolder
- removed H1, H2, H3, H4, H5: MountingHole, MountingHole:MountingHole_2.2mm_M2_DIN965_Pad
- removed R10: 1k5, Resistor_SMD:R_0402_1005Metric
- removed R24, R25: 1.5k, LED_SMD:LED_0805_2012Metric_Pad1.15x1.40mm_HandSolder
- added C19: 10u, Capacitor_Tantalum_SMD:CP_EIA-3216-18_Kemet-A_Pad1.58x1.35mm_HandSolder, B.Cu at (258.4, 117.2)
- added C5: 0.1u, Capacitor_SMD:C_0805_2012Metric_Pad1.18x1.45mm_HandSolder, B.Cu at (246.5, 103.2)
- added C6: 10u, Capacitor_Tantalum_SMD:CP_EIA-3216-18_Kemet-A_Pad1.58x1.35mm_HandSolder, B.Cu at (265.2, 120.4)
- added D30: Schottky, Diode_SMD:D_SOD-123, B.Cu at (260.1, 107.2)
- added J2: USB_C_Receptacle_USB2.0_16P, reversible_skyline:USB_C_Receptacle_HRO_TYPE-C-31-M-12_reversible, F.Cu at (262.8, 76.7)
- added MH1: MountingHole, , F.Cu at (139.6, 97.6)
- added MH2: MountingHole, , F.Cu at (215.6, 96.5)
- added MH3: , ceoloide:mounting_hole_npth, F.Cu at (215.6, 132.4)
- added MH4: , ceoloide:mounting_hole_npth, F.Cu at (139.6, 136.0)
- added MH5: MountingHole, , F.Cu at (250.2, 152.6)
- added R28: 0R, Resistor_SMD:R_0805_2012Metric_Pad1.20x1.40mm_HandSolder, B.Cu at (256.0, 122.6)
- added R31: 0R, Resistor_SMD:R_0805_2012Metric_Pad1.20x1.40mm_HandSolder, B.Cu at (259.0, 122.6)
- C12, C13, C14, C15, C16, C36, C37, C7: footprint Capacitor_SMD:C_0402_1005Metric -> Capacitor_SMD:C_0805_2012Metric_Pad1.18x1.45mm_HandSolder; moved to B.Cu
- D1, D10, D11, D12, D13, D14, D15, D16, D17, D18, D19, D2, D20, D21, D22, D23, D24, D25, D26, D27, D28, D3, D4, D5, D6, D7, D8, D9: footprint reversible_skyline:reversible_D_0805_2012Metric_Pad1.15x1.40mm_HandSolder -> reversible_skyline:designator_swapped_D_0805_2012Metric_Pad1.15x1.40mm_HandSolder; moved to B.Cu
- D31, F2, JP10, JP6, JP7, JP8, JP9, Q3, Q5, Q6, R27, U10, U4, U7: moved to B.Cu
- J5: footprint Connector_PinHeader_2.54mm:PinHeader_1x05_P2.54mm_Vertical -> Connector_IDC:IDC-Header_2x03_P2.54mm_Vertical_SMD
- J7: footprint PCM_marbastlib-various:Molex_Pico-EZmate_78171-0002_1x02-1MP_P1.20mm_Vertical -> reversible_skyline:reversible_Molex_Pico-EZmate_78171-0002_1x02-1MP_P1.20mm_Vertical
- R1, R11, R12, R13, R14, R19, R2, R20, R21, R5, R6, R7, R8: footprint LED_SMD:LED_0805_2012Metric_Pad1.15x1.40mm_HandSolder -> Resistor_SMD:R_0805_2012Metric_Pad1.20x1.40mm_HandSolder; moved to B.Cu
- R15, R16, R22, R23, R29, R30, R9: footprint Resistor_SMD:R_0402_1005Metric -> Resistor_SMD:R_0805_2012Metric_Pad1.20x1.40mm_HandSolder; moved to B.Cu
- R17, R18: footprint Resistor_SMD:R_0603_1608Metric_Pad0.98x0.95mm_HandSolder -> Resistor_SMD:R_0805_2012Metric_Pad1.20x1.40mm_HandSolder; moved to B.Cu
- R3, R4: footprint Resistor_SMD:R_0402_1005Metric_Pad0.72x0.64mm_HandSolder -> Resistor_SMD:R_0805_2012Metric_Pad1.20x1.40mm_HandSolder; moved to B.Cu
- S1, S10, S11, S12, S13, S14, S15, S16, S17, S18, S19, S2, S20, S21, S22, S23, S24, S25, S26, S27, S28, S3, S4, S5, S6, S7, S8, S9: value choc_v1_SW_solder -> MX_SW_solder; footprint PCM_marbastlib-xp-choc:SW_choc_Reversible_1u -> PCM_marbastlib-xp-mx:SW_MX_Reversible_1u
- SW4: footprint PCM_marbastlib-various:SW_SPST_SKQG_WithStem -> reversible_skyline:reversible_SW_SPST_SKQG_WithStem
- SW7: footprint PCM_marbastlib-various:SW_MSK12C02-HB -> PCM_marbastlib-various:reversible_SW_MSK12C02-HB
- U5: footprint PCM_marbastlib-various:nRF52840_holyiot_18010 -> reversible_skyline:nRF52840_holyiot_18010_HS_simple_reversible
- moved R13 216.9 mm to (139.5, 143.9)
- moved R5 212.4 mm to (139.4, 89.9)
- moved R8 210.6 mm to (139.5, 121.8)
- moved D41 182.6 mm to (139.5, 141.0)
- moved D38 180.2 mm to (139.5, 118.0)
- moved R14 177.8 mm to (177.4, 133.1)
- moved R11 177.2 mm to (177.7, 114.5)
- moved D35 174.9 mm to (139.5, 93.5)
- moved R6 174.4 mm to (177.4, 95.6)
- moved R2 157.8 mm to (197.2, 154.1)
- moved R29 143.0 mm to (235.9, 123.2), turned to 180 degrees
- moved D42 142.9 mm to (177.5, 130.5)
- moved D39 141.3 mm to (177.8, 111.8)
- moved R20 140.7 mm to (217.7, 158.4), turned to 170 degrees
- moved R19 140.2 mm to (215.5, 139.2)
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Connections:
- net Case renamed GND
- net LED_PWR renamed LED_Pwr
- JP9 pad 2: unconnected-(JP9-B-Pad2) -> Net-(JP4-B)
- U10 pad 6: Net-(U10-STDBY) -> unconnected-(U10-STDBY-Pad6)
- U5 pad 18: unconnected-(U5-P0.23-Pad18) -> EncoderTermA
- U5 pad 19: unconnected-(U5-P0.21-Pad19) -> EncoderTermB
- U5 pad 20: unconnected-(U5-P0.19-Pad20) -> COL5
- U5 pad 26: unconnected-(U5-P0.22-Pad26) -> COL4
- U5 pad 27: unconnected-(U5-P1.00-Pad27) -> COL3
- U5 pad 28: unconnected-(U5-P1.03-LF-Pad28) -> COL2
- U5 pad 29: unconnected-(U5-P1.01-LF-Pad29) -> COL1
- U5 pad 30: unconnected-(U5-P1.02-LF-Pad30) -> COL0
- U5 pad 31: unconnected-(U5-SWDCLK-Pad31) -> SWDCLK
- U5 pad 32: unconnected-(U5-SWDIO-Pad32) -> SWDIO
- U5 pad 33: unconnected-(U5-P1.04-LF-Pad33) -> MOSI
- U5 pad 34: unconnected-(U5-P1.06-LF-Pad34) -> SCK
- U5 pad 4: unconnected-(U5-P1.13-LF-Pad4) -> CS
- U5 pad 5: unconnected-(U5-P1.15-LF-Pad5) -> LED_Ctrl
Routing:
- net LED_Pwr: track 0.00 -> 360.4 mm, vias 0 -> 16
- net COL2: track 0.00 -> 209.2 mm, vias 0 -> 3
- net COL0: track 0.00 -> 204.1 mm, vias 0 -> 1
- net COL3: track 0.00 -> 189.4 mm, vias 0 -> 4
- net COL1: track 0.00 -> 185.6 mm, vias 0 -> 2
- net COL4: track 0.00 -> 179.0 mm, vias 0 -> 5
- net ROW4: track 0.00 -> 172.7 mm, vias 0 -> 10
- net ROW3: track 0.00 -> 170.0 mm, vias 0 -> 6
- net ROW2: track 0.00 -> 158.8 mm, vias 0 -> 4
- net ROW1: track 0.00 -> 141.9 mm, vias 0 -> 4
- net ROW0: track 0.00 -> 137.8 mm, vias 0 -> 2
- net COL5: track 0.00 -> 129.3 mm, vias 0 -> 5
- net +3.3V: track 0.00 -> 123.9 mm, vias 0 -> 11
- net +5V: track 0.00 -> 115.2 mm, vias 0 -> 12
- net SWDCLK: track 0.00 -> 99.2 mm, vias 0 -> 3
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- added copper zone on B.Cu, net GND
- added copper zone on F.Cu, net GND
Other:
- board size 140.5 x 109.7 mm -> 151 x 125.6 mm

Commit message: finished routing, need to review
Parts:
- removed J5: Conn_01x05, Connector_IDC:IDC-Header_2x03_P2.54mm_Vertical_SMD
- added J1: wurth_6_pin_SKEDD, 490107670612:wurth_6_pin_SKEDD, F.Cu at (264.7, 147.5)
- D1, D10, D11, D12, D13, D14, D15, D16, D17, D18, D19, D2, D20, D21, D22, D23, D24, D25, D26, D27, D28, D3, D4, D5, D6, D7, D8, D9: footprint reversible_skyline:designator_swapped_D_0805_2012Metric_Pad1.15x1.40mm_HandSolder -> Diode_SMD:D_0805_2012Metric_Pad1.15x1.40mm_HandSolder
- MH1: value MountingHole -> MH1; footprint (none) -> reversible_skyline:mounting_hole_npth
- MH2: value MountingHole -> MH2; footprint (none) -> reversible_skyline:mounting_hole_npth
- MH3: value (none) -> MH3; footprint ceoloide:mounting_hole_npth -> reversible_skyline:mounting_hole_npth
- MH4: value (none) -> MH4; footprint ceoloide:mounting_hole_npth -> reversible_skyline:mounting_hole_npth
- MH5: value MountingHole -> MH5; footprint (none) -> reversible_skyline:mounting_hole_npth
- moved MH2 85.6 mm to (139.6, 136.0)
- moved MH4 76.1 mm to (215.6, 132.4)
- moved MH3 35.9 mm to (215.6, 96.5)
- moved C36 18.2 mm to (236.2, 96.8), turned to -90 degrees
- moved C37 16.6 mm to (253.5, 96.2)
- moved JP10 10.2 mm to (250.5, 107.0)
- moved JP6 10.2 mm to (240.2, 107.0)
- moved JP9 5.00 mm to (247.8, 107.0)
- moved JP7 5.00 mm to (242.8, 107.0)
- moved R18 2.52 mm to (236.4, 140.4)
- moved D28 2.21 mm to (259.6, 128.4)
- moved R17 1.92 mm to (259.0, 141.2), turned to 90 degrees
- moved R30 1.45 mm to (239.5, 120.8)
- moved C14 1.18 mm to (258.8, 100.0), turned to 0 degrees
- moved C5 1.07 mm to (247.0, 102.3)
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Connections:
- U5 pad 10: ROW4 -> COL3
- U5 pad 11: Vsense -> COL4
- U5 pad 12: Vsense_EN -> COL5
- U5 pad 17: unconnected-(U5-P0.12-Pad17) -> MOSI
- U5 pad 18: EncoderTermA -> SCK
- U5 pad 19: EncoderTermB -> CS
- U5 pad 2: unconnected-(U5-P1.11-LF-Pad2)_1 -> ROW0
- U5 pad 20: COL5 -> unconnected-(U5-P0.19-Pad20)
- U5 pad 26: COL4 -> Vsense
- U5 pad 27: COL3 -> Vsense_EN
- U5 pad 28: COL2 -> LED_Ctrl
- U5 pad 29: COL1 -> EncoderTermB
- U5 pad 3: unconnected-(U5-P1.10-LF-Pad3)_1 -> ROW1
- U5 pad 30: COL0 -> EncoderTermA
- U5 pad 33: MOSI -> unconnected-(U5-P1.04-LF-Pad33)_1
- U5 pad 34: SCK -> unconnected-(U5-P1.06-LF-Pad34)_1
- U5 pad 4: CS -> ROW2
- U5 pad 5: LED_Ctrl -> ROW3
- U5 pad 6: ROW0 -> ROW4
- U5 pad 7: ROW1 -> COL0
- U5 pad 8: ROW2 -> COL1
- U5 pad 9: ROW3 -> COL2
Routing:
- net EncoderTermB: track 62.2 -> 88.3 mm, vias 2 -> 4
- net LED_Pwr: track 360.4 -> 386.0 mm
- net SCK: track 52.2 -> 27.4 mm, vias 6 -> 4
- net MOSI: track 50.9 -> 31.1 mm, vias 5 -> 4
- net Net-(JP1-B): track 23.5 -> 5.09 mm, vias 1 -> 0
- net GND: track 86.7 -> 104.5 mm, vias 36 -> 37
- net CS: track 42.5 -> 25.3 mm, vias 5 -> 4
- net Net-(JP10-B): track 21.0 -> 5.16 mm, vias 1 -> 0
- net RST: track 70.4 -> 83.8 mm, vias 7 -> 5
- net ROW3: track 170.0 -> 182.4 mm, vias 6 -> 4
- net EncoderTermA: track 71.3 -> 82.3 mm, vias 4 -> 3
- net Net-(JP4-B): track 15.3 -> 5.05 mm
- net ROW2: track 158.8 -> 168.7 mm
- net Net-(R23-Pad2): track 49.7 -> 39.8 mm
- net COL1: track 185.6 -> 176.1 mm, vias 2 -> 5
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